File: PCB/NODE_DATAPAC_128K_256K.kicad_pcb (KiCad board)
At the start: 2 copper layers, 254 x 43.2 mm, 20 parts, among them J1 Conn_02x20_Odd_Even, U1 74161, U10/U14 62256, U2 74161, U3 74161, U4 74138, U5 74138, U6 74374, U7/U11 62256, U8/U12 62256, U9/U13 62256

Commit message: WIP: PCB
Parts:
- added TP5: VMEM+, 000_LOCAL:TP_THT_pwr, F.Cu at (210.8, 85.2)
- added TP6: VMEM-, 000_LOCAL:TP_THT_pwr, F.Cu at (210.8, 89.5)
- U10/U14, U7/U11, U8/U12, U9/U13: value 62256 -> 62256-DIP
- moved R3 10.1 mm to (34.3, 123.2), turned to 0 degrees
- moved R2 10.1 mm to (47.0, 123.2), turned to 0 degrees
- moved J1 6.35 mm to (142.2, 118.6)
- moved U5 0.51 mm to (34.3, 118.1)
Connections:
- J1 pad 2: unconnected-(J1-Pin_2-Pad2) -> VBUS
Routing:
- net GND: track 0.00 -> 424.3 mm, vias 0 -> 4
- net Net-(U1-CP): track 0.00 -> 330.5 mm, vias 0 -> 1
- net VBUS: track 0.00 -> 320.2 mm, vias 0 -> 3
- net VMEM: track 0.00 -> 271.6 mm
- net Net-(U5-A1): track 0.00 -> 190.9 mm, vias 0 -> 1
- net /~{BANK0_0}: track 0.00 -> 174.8 mm
- net Net-(U1-~{MR}): track 0.00 -> 115.4 mm, vias 0 -> 1
- net /A8: track 0.00 -> 108.0 mm, vias 0 -> 1
- net /AD1: track 0.00 -> 79.1 mm
- net /~{RD}: track 0.00 -> 79.0 mm, vias 0 -> 1
- net /~{BANK1_3}: track 0.00 -> 52.5 mm
- net Net-(U2-CEP): track 0.00 -> 35.1 mm, vias 0 -> 1
- net Net-(U5-A0): track 0.00 -> 26.9 mm, vias 0 -> 1
- net Net-(U1-CEP): track 0.00 -> 25.5 mm
- net Net-(BT1-+): track 0.00 -> 25.4 mm
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
Commit message: PCB!
Parts:
- U10/U14, U7/U11, U8/U12, U9/U13: value 62256-DIP -> 62256
- moved U1 1.27 mm to (261.6, 113.3)
Routing:
- net /~{WR}: track 0.00 -> 266.9 mm, vias 0 -> 1
- net Net-(U1-Q0): track 0.00 -> 262.7 mm
- net Net-(U1-Q1): track 0.00 -> 240.0 mm
- net /AD0: track 0.00 -> 231.7 mm, vias 0 -> 3
- net /AD6: track 0.00 -> 229.1 mm, vias 0 -> 2
- net /AD7: track 0.00 -> 221.8 mm, vias 0 -> 2
- net /AD4: track 0.00 -> 211.5 mm, vias 0 -> 3
- net /AD5: track 0.00 -> 206.1 mm, vias 0 -> 1
- net /AD2: track 0.00 -> 203.5 mm, vias 0 -> 3
- net Net-(U10/U14-A8): track 0.00 -> 201.6 mm
- net Net-(U10/U14-A9): track 0.00 -> 195.4 mm
- net Net-(U10/U14-A4): track 0.00 -> 192.3 mm
- net Net-(U10/U14-A3): track 0.00 -> 192.3 mm
- net Net-(U10/U14-A2): track 0.00 -> 192.3 mm
- net Net-(U10/U14-A1): track 0.00 -> 192.3 mm
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
Commit message: optimize some traces
Parts:
- moved TP6 0.13 mm to (210.8, 89.4)
Connections:
- U1 pad 3: unconnected-(U1-D0-Pad3) -> GND
- U1 pad 4: unconnected-(U1-D1-Pad4) -> GND
- U1 pad 5: unconnected-(U1-D2-Pad5) -> GND
- U1 pad 6: unconnected-(U1-D3-Pad6) -> GND
- U2 pad 3: unconnected-(U2-D0-Pad3) -> GND
- U2 pad 4: unconnected-(U2-D1-Pad4) -> GND
- U2 pad 5: unconnected-(U2-D2-Pad5) -> GND
- U2 pad 6: unconnected-(U2-D3-Pad6) -> GND
- U3 pad 3: unconnected-(U3-D0-Pad3) -> GND
- U3 pad 4: unconnected-(U3-D1-Pad4) -> GND
- U3 pad 5: unconnected-(U3-D2-Pad5) -> GND
- U3 pad 6: unconnected-(U3-D3-Pad6) -> GND
Routing:
- net GND: track 424.6 -> 0.00 mm, vias 4 -> 46
- net /~{WR}: track 266.9 -> 157.5 mm
- net /~{BANK1_3}: track 52.5 -> 30.2 mm
- net /~{RD}: track 164.9 -> 158.2 mm, vias 1 -> 0
- net Net-(U5-A2): track 175.2 -> 170.8 mm
- net Net-(U5-A0): track 171.7 -> 167.4 mm
- net /~{BANK0_3}: track 24.6 -> 28.5 mm
- net Net-(U1-Q0): track 262.7 -> 259.6 mm
- net /AD6: track 229.1 -> 226.6 mm
- net VBUS: track 316.6 -> 319.0 mm
- net /~{BANK0_1}: track 120.3 -> 118.3 mm
- net /~{BANK1_1}: track 109.1 -> 107.1 mm
- net /AD0: track 231.7 -> 229.8 mm
- net VMEM: track 270.2 -> 268.3 mm
- net /~{BANK1_0}: track 150.6 -> 149.2 mm
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- added copper zone on B.Cu, net GND
- added copper zone on F.Cu, net GND
Other:
- board text added: "${TITLE} - v${REVISION} ${COMMENT1}"
- board text added: "A10"
- board text added: "A11"
- board text added: "A12"
- board text added: "A13"
- board text added: "A14"
- board text added: "A15"
- board text added: "A8"
- board text added: "A9"
- board text added: "AD0"
- board text added: "AD1"
- board text added: "AD2"
- board text added: "AD3"
- board text added: "AD4"
- board text added: "AD5"
- board text added: "AD6"
- board text added: "AD7"
- board text added: "CLK"
- board text added: "GND"
- board text added: "INTR"
- board text added: "IO/~{M}"
- board text added: "RAM_RST"
- board text added: "S0"
- board text added: "S1"
- board text added: "VCC"
- board text added: "Y0"
- board text added: "nc"
- board text added: "~{ALE}"
- board text added: "~{A}"
- board text added: "~{RD}"
- board text added: "~{RESET}"
- board text added: "~{WR}"

Commit message: silkscreen
Routing:
- net Net-(U1-Q0): track 259.6 -> 259.0 mm
- net VBUS: track 319.0 -> 319.5 mm
Other:
- board text added: "NODE DATAPAC 256K REPRODUCTION"
