File: PCB/MiniNDP_256.kicad_sch (KiCad schematic)
At the start: 18 parts, among them J1 Conn_02x20_Odd_Even, U1 74161, U2 74161, U3 74161, U4 74138, U5 74374, U6 AS6C2008A, U7 74LVC1G32

Commit message: MiniNDP
Parts:
- removed R1: 5.1k, 000_LOCAL:R_0805, symbol 000_LOCAL:R
- added C6: 47u, 000_LOCAL:C_1206, symbol 000_LOCAL:C
- U7: value 74LVC1G32 -> 741G32
Connections:
- net GND: now also C6.2
- net SLEEP: now also D2.2 (A); no longer D2.1 (A)
- net VBUS: now also C6.1
Other:
- note added: "+3VDC"
- note added: "AS6C2008A is optimal, but AS6C4008 is also compatible. With AS6C4008 installed: Pin 6 is A17, high at all times, essentially inert, pin 9 is A18, receiving/returning the A17 data, resulting in the same outward functionality."
- note added: "SYSTEM BUS connection is using STANDARD pin numbering for the connector, NOT the odd<>even swapped numbering from the TANDY Model 102 & 200 manuals. Example, RAM_RST is actually on pin 38, but the TANDY 102 & 200 manuals call it pin 37."
- note removed: "A 256Kx8 SRAM (AS6C2008A) is optimal, but those are rare now. U6 shows the pinout for AS6C2008A, but AS6C4008 is also compatible, even though the pinout is different. With AS6C4008 installed: Pin 6 is A17, high at all times, essentially inert, pin 9 is A18, receiving/returning the A17 data, resulting in the same outward functionality. The fast-disable-on-disconnect behavior to protect data from b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"
- note removed: "ON"
- note removed: "SYSTEM BUS connection here is using the standard pin numbering for the connector, NOT the odd/even swapped numbering from the TANDY Model 102 & 200 manuals. Example, RAM_RST is actually on pin 38, but the TANDY 102 & 200 manuals call it pin 37."
- title: NODE DATAPAC 256K bkw0 -> MiniNDP_256

Commit message: MiniNDP sch
Connections:
- no-connect marks 26 -> 27
Other:
- title: MiniNDP_256 -> MiniNDP 256
Changed lines of the file:
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@@
   (paper "A3")
   (title_block
-    (title "MiniNDP_256")
+    (title "MiniNDP 256")
     (date "2023-08-28")
     (rev "001")
@@
   (no_connect (at 109.22 175.26))
   (no_connect (at 109.22 182.88))
+  (no_connect (at 133.35 200.66))
   (no_connect (at 96.52 160.02))
   (no_connect (at 114.3 77.47))
@@
     (stroke (width 0) (type default))
   )
-  (bus_entry (at 346.71 85.09) (size 2.54 -2.54)
+  (bus_entry (at 340.36 85.09) (size 2.54 -2.54)
     (stroke (width 0) (type default))
   )
@@
     (stroke (width 0) (type default))
   )
-  (bus_entry (at 346.71 92.71) (size 2.54 -2.54)
+  (bus_entry (at 340.36 92.71) (size 2.54 -2.54)
     (stroke (width 0) (type default))
   )
@@
     (stroke (width 0) (type default))
   )
-  (bus_entry (at 346.71 95.25) (size 2.54 -2.54)
+  (bus_entry (at 340.36 95.25) (size 2.54 -2.54)
     (stroke (width 0) (type default))
   )
@@
     (stroke (width 0) (type default))
   )
-  (bus_entry (at 346.71 100.33) (size 2.54 -2.54)
-    (stroke (width 0) (type default))
-  )
-  (bus_entry (at 346.71 97.79) (size 2.54 -2.54)
+  (bus_entry (at 340.36 100.33) (size 2.54 -2.54)
+    (stroke (width 0) (type default))
+  )
+  (bus_entry (at 340.36 97.79) (size 2.54 -2.54)
     (stroke (width 0) (type default))
   )
@@
     (stroke (width 0) (type default))
   )
-  (bus_entry (at 346.71 87.63) (size 2.54 -2.54)
-    (stroke (width 0) (type default))
-  )
-  (bus_entry (at 346.71 125.73) (size 2.54 -2.54)
-    (stroke (width 0) (type default))
-  )
-  (bus_entry (at 346.71 123.19) (size 2.54 -2.54)
+  (bus_entry (at 340.36 87.63) (size 2.54 -2.54)
+    (stroke (width 0) (type default))
+  )
+  (bus_entry (at 340.36 125.73) (size 2.54 -2.54)
+    (stroke (width 0) (type default))
+  )
+  (bus_entry (at 340.36 123.19) (size 2.54 -2.54)
     (stroke (width 0) (type default))
   )
@@
     (stroke (width 0) (type default))
   )
-  (bus_entry (at 346.71 82.55) (size 2.54 -2.54)
+  (bus_entry (at 340.36 82.55) (size 2.54 -2.54)
     (stroke (width 0) (type default))
   )
@@
     (stroke (width 0) (type default))
   )
-  (bus_entry (at 346.71 90.17) (size 2.54 -2.54)
+  (bus_entry (at 340.36 90.17) (size 2.54 -2.54)
     (stroke (width 0) (type default))
   )
@@
     (stroke (width 0) (type default))
   )
-  (wire (pts (xy 342.9 118.11) (xy 330.2 118.11))
+  (wire (pts (xy 337.82 118.11) (xy 330.2 118.11))
     (stroke (width 0) (type default))
   )
@@
     (stroke (width 0) (type default))
   )
+  (bus (pts (xy 342.9 97.79) (xy 342.9 120.65))
+    (stroke (width 0) (type default))
+  )
   (wire (pts (xy 234.95 97.79) (xy 245.11 97.79))
     (stroke (width 0) (type default))
@@
     (stroke (width 0) (type default))
   )
-  (wire (pts (xy 330.2 100.33) (xy 346.71 100.33))
+  (wire (pts (xy 330.2 100.33) (xy 340.36 100.33))
     (stroke (width 0) (type default))
   )
@@
     (stroke (width 0) (type default))
   )
-  (wire (pts (xy 330.2 182.88) (xy 342.9 182.88))
+  (wire (pts (xy 330.2 182.88) (xy 337.82 182.88))
     (stroke (width 0) (type default))
   )
@@
     (stroke (width 0) (type default))
   )
-  (bus (pts (xy 349.25 90.17) (xy 349.25 92.71))
-    (stroke (width 0) (type default))
-  )
-  (wire (pts (xy 330.2 95.25) (xy 346.71 95.25))
+  (bus (pts (xy 342.9 90.17) (xy 342.9 92.71))
+    (stroke (width 0) (type default))
+  )
+  (wire (pts (xy 330.2 95.25) (xy 340.36 95.25))
     (stroke (width 0) (type default))
   )
@@
     (stroke (width 0) (type default))
   )
-  (bus (pts (xy 349.25 92.71) (xy 349.25 95.25))
+  (bus (pts (xy 342.9 92.71) (xy 342.9 95.25))
     (stroke (width 0) (type default))
   )
@@
     (stroke (width 0) (type default))
   )
-  (bus (pts (xy 349.25 85.09) (xy 349.25 87.63))
+  (bus (pts (xy 342.9 85.09) (xy 342.9 87.63))
     (stroke (width 0) (type default))
   )
@@
     (stroke (width 0) (type default))
   )
-  (wire (pts (xy 330.2 90.17) (xy 346.71 90.17))
+  (wire (pts (xy 330.2 90.17) (xy 340.36 90.17))
     (stroke (width 0) (type default))
   )
@@
     (stroke (width 0) (type default))
   )
-  (wire (pts (xy 330.2 123.19) (xy 346.71 123.19))
-    (stroke (width 0) (type default))
-  )
-  (bus (pts (xy 349.25 120.65) (xy 349.25 123.19))
+  (wire (pts (xy 330.2 123.19) (xy 340.36 123.19))
+    (stroke (width 0) (type default))
+  )
+  (bus (pts (xy 342.9 120.65) (xy 342.9 123.19))
     (stroke (width 0) (type default))
   )
@@
     (stroke (width 0) (type default))
   )
-  (bus (pts (xy 349.25 82.55) (xy 349.25 85.09))
+  (bus (pts (xy 342.9 82.55) (xy 342.9 85.09))
     (stroke (width 0) (type default))
   )
@@
     (stroke (width 0) (type default))
   )
-  (bus (pts (xy 349.25 95.25) (xy 349.25 97.79))
+  (bus (pts (xy 342.9 95.25) (xy 342.9 97.79))
     (stroke (width 0) (type default))
   )
@@
     (stroke (width 0) (type default))
   )
-  (bus (pts (xy 349.25 80.01) (xy 349.25 82.55))
+  (bus (pts (xy 342.9 80.01) (xy 342.9 82.55))
     (stroke (width 0) (type default))
   )
@@
     (stroke (width 0) (type default))
   )
-  (wire (pts (xy 330.2 92.71) (xy 346.71 92.71))
+  (wire (pts (xy 330.2 92.71) (xy 340.36 92.71))
     (stroke (width 0) (type default))
   )
@@
     (stroke (width 0) (type default))
   )
-  (bus (pts (xy 165.1 203.2) (xy 349.25 203.2))
+  (bus (pts (xy 165.1 203.2) (xy 342.9 203.2))
     (stroke (width 0) (type default))
   )
@@
     (stroke (width 0) (type default))
   )
-  (bus (pts (xy 349.25 87.63) (xy 349.25 90.17))
+  (bus (pts (xy 342.9 87.63) (xy 342.9 90.17))
     (stroke (width 0) (type default))
   )
@@
     (stroke (width 0) (type default))
   )
-  (wire (pts (xy 330.2 87.63) (xy 346.71 87.63))
+  (wire (pts (xy 330.2 87.63) (xy 340.36 87.63))
     (stroke (width 0) (type default))
   )
@@
     (stroke (width 0) (type default))
   )
-  (wire (pts (xy 330.2 85.09) (xy 346.71 85.09))
-    (stroke (width 0) (type default))
-  )
-  (wire (pts (xy 330.2 82.55) (xy 346.71 82.55))
+  (wire (pts (xy 330.2 85.09) (xy 340.36 85.09))
+    (stroke (width 0) (type default))
+  )
+  (wire (pts (xy 330.2 82.55) (xy 340.36 82.55))
     (stroke (width 0) (type default))
   )
@@
     (stroke (width 0) (type default))
   )
-  (wire (pts (xy 330.2 97.79) (xy 346.71 97.79))
+  (wire (pts (xy 330.2 97.79) (xy 340.36 97.79))
     (stroke (width 0) (type default))
   )
@@
     (stroke (width 0) (type default))
   )
-  (wire (pts (xy 342.9 182.88) (xy 342.9 118.11))
+  (wire (pts (xy 337.82 182.88) (xy 337.82 118.11))
     (stroke (width 0) (type default))
   )
@@
     (stroke (width 0) (type default))
   )
-  (bus (pts (xy 349.25 97.79) (xy 349.25 120.65))
-    (stroke (width 0) (type default))
-  )
   (wire (pts (xy 294.64 125.73) (xy 304.8 125.73))
     (stroke (width 0) (type default))
@@
     (stroke (width 0) (type default))
   )
-  (bus (pts (xy 349.25 123.19) (xy 349.25 203.2))
+  (bus (pts (xy 342.9 123.19) (xy 342.9 203.2))
     (stroke (width 0) (type default))
   )
@@
     (stroke (width 0) (type default))
   )
-  (wire (pts (xy 330.2 125.73) (xy 346.71 125.73))
+  (wire (pts (xy 330.2 125.73) (xy 340.36 125.73))
     (stroke (width 0) (type default))
   )
@@
     (effects (font (size 1.27 1.27)) (justify right bottom))
   )
+  (label "RAM_RST" (at 128.27 193.04 180) (fields_autoplaced)
+    (effects (font (size 1.27 1.27)) (justify right bottom))
+  )
   (label "AD6" (at 96.52 154.94 180) (fields_autoplaced)
     (effects (font (size 1.27 1.27)) (justify right bottom))
@@
     (effects (font (size 1.27 1.27)) (justify left bottom))
   )
+  (label "SLEEP" (at 133.35 185.42 0) (fields_autoplaced)
+    (effects (font (size 1.27 1.27)) (justify left bottom))
+  )

Commit message: datasheets, battery holder
Parts:
- BT1: footprint 000_LOCAL:BatteryHolder_Keystone_3034_1x20mm -> 000_LOCAL:CR2032_holder_Keystone_3034
Changed lines of the file:
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@@
       (effects (font (size 1.27 1.27)) hide)
     )
-    (property "Datasheet" "https://www.alliancememory.com/wp-content/uploads/pdf/AS6C4008.pdf" (at 317.5 104.14 0)
+    (property "Datasheet" "datasheets/AS6C4008.pdf" (at 317.5 104.14 0)
       (effects (font (size 1.27 1.27)) hide)
     )
@@
       (effects (font (size 1.27 1.27)))
     )
-    (property "Footprint" "000_LOCAL:BatteryHolder_Keystone_3034_1x20mm" (at 234.95 263.906 90)
-      (effects (font (size 1.27 1.27)) hide)
-    )
-    (property "Datasheet" "~" (at 234.95 263.906 90)
-      (effects (font (size 1.27 1.27)) hide)
-    )
+    (property "Footprint" "000_LOCAL:CR2032_holder_Keystone_3034" (at 234.95 263.906 90)
+      (effects (font (size 1.27 1.27)) hide)
+    )
+    (property "Datasheet" "datasheets/Keystone_3034.pdf" (at 234.95 263.906 90)
+      (effects (font (size 1.27 1.27)) hide)
+    )

Commit message: sch slight tidy
Other:
- note added: "AS6C2008A (256Kx8) or AS6C4008 (512Kx8)"
- note removed: "AS6C2008A (256Kx8) or AS6C4008 (512Kx8) or equivalents"
Changed lines of the file:
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@@
   )
   (text "\nAS6C2008A is optimal, but AS6C4008 is also compatible.\n\nWith AS6C4008 installed:\nPin 6 is A17, high at all times, essentially inert,\npin 9 is A18, receiving/returning the A17 data,\nresulting in the same outward functionality.\n"
-    (at 279.4 52.07 0)
+    (at 280.67 60.96 0)
     (effects (font (size 2 2)) (justify left bottom))
   )
@@
     (effects (font (size 1.27 1.27)) (justify right bottom))
   )
-  (text "AS6C2008A (256Kx8)\nor AS6C4008 (512Kx8)\nor equivalents"
-    (at 300.99 71.12 0)
+  (text "AS6C2008A (256Kx8)\nor AS6C4008 (512Kx8)" (at 300.99 71.12 0)
     (effects (font (size 2 2)) (justify left bottom))
   )
@@
   )
   (text "Each ~{BLOCK} pulse updates local A10-A17 from BUS AD0-AD7 and resets the byte counter to 0.\n\nEach ~{BYTE} pulse disables SRAM, advances the byte counter by 1, and sets local A0-A9.\n\n8 bits from the bus = 256 possible block-start addresses from the bus.\n10 bits byte counter = 1k per block."
-    (at 62.23 241.3 0)
+    (at 31.75 266.7 0)
     (effects (font (size 1.27 1.27)) (justify left bottom))
   )
@@
     (effects (font (size 1.27 1.27)) (justify left bottom))
   )
-  (text "(AS6C4008)" (at 312.42 106.68 0)
+  (text "(AS6C4008)" (at 331.47 78.74 0)
     (effects (font (size 1.27 1.27)) (justify left bottom))
   )
@@
   (symbol (lib_id "000_LOCAL:AS6C2008_TSOP-I-32") (at 317.5 101.6 0) (unit 1)
     (in_bom yes) (on_board yes) (dnp no)
-    (property "Reference" "U6" (at 307.34 78.105 0)
-      (effects (font (size 1.27 1.27)) (justify left bottom))
-    )
-    (property "Value" "AS6C2008A" (at 317.5 104.14 0)
-      (effects (font (size 1.27 1.27)) (justify bottom))
+    (property "Reference" "U6" (at 320.04 74.93 0)
+      (effects (font (size 1.27 1.27)) (justify left))
+    )
+    (property "Value" "AS6C2008A" (at 320.04 77.47 0)
+      (effects (font (size 1.27 1.27)) (justify left))
     )
     (property "Footprint" "000_LOCAL:TSOP32-dual" (at 317.5 101.6 0)
@@
       (effects (font (size 1.27 1.27)) hide)
     )
-    (property "Value" "VMEM" (at 317.5 167.64 0)
+    (property "Value" "VMEM" (at 313.69 170.18 0)
       (effects (font (size 1.27 1.27)))
     )
@@
       (effects (font (size 1.27 1.27)) hide)
     )
-    (property "Value" "VMEM" (at 220.98 251.46 0)
+    (property "Value" "VMEM" (at 220.98 250.19 0)
       (effects (font (size 1.27 1.27)))
     )
@@
   )
   (symbol (lib_id "power:GND") (at 101.6 102.87 0) (unit 1)
-    (in_bom yes) (on_board yes) (dnp no) (fields_autoplaced)
+    (in_bom yes) (on_board yes) (dnp no)
     (property "Reference" "#PWR022" (at 101.6 109.22 0)
       (effects (font (size 1.27 1.27)) hide)
     )
-    (property "Value" "GND" (at 101.6 107.95 0)
+    (property "Value" "GND" (at 97.79 105.41 0)
       (effects (font (size 1.27 1.27)))
     )
@@
       (effects (font (size 1.27 1.27)) hide)
     )
-    (property "Value" "VMEM" (at 317.5 73.66 0)
+    (property "Value" "VMEM" (at 313.69 74.93 0)
       (effects (font (size 1.27 1.27)))
     )
@@
       (effects (font (size 1.27 1.27)) hide)
     )
-    (property "Value" "GND" (at 190.5 114.3 0)
+    (property "Value" "GND" (at 186.69 111.76 0)
       (effects (font (size 1.27 1.27)))
     )
@@
       (effects (font (size 1.27 1.27)) hide)
     )
-    (property "Value" "GND" (at 317.5 135.89 0)
+    (property "Value" "GND" (at 313.69 133.35 0)
       (effects (font (size 1.27 1.27)))
     )
@@
       (effects (font (size 1.27 1.27)) hide)
     )
-    (property "Value" "VMEM" (at 133.35 172.72 0)
+    (property "Value" "VMEM" (at 133.35 173.99 0)
       (effects (font (size 1.27 1.27)))
     )
@@
       (effects (font (size 1.27 1.27)) hide)
     )
-    (property "Value" "GND" (at 158.75 92.71 0)
+    (property "Value" "GND" (at 154.94 90.17 0)
       (effects (font (size 1.27 1.27)))
     )
@@
       (effects (font (size 1.27 1.27)) hide)
     )
-    (property "Value" "VBUS" (at 213.36 256.54 0)
+    (property "Value" "VBUS" (at 213.36 255.27 0)
       (effects (font (size 1.27 1.27)))
     )
@@
       (effects (font (size 1.27 1.27)) hide)
     )
-    (property "Value" "GND" (at 222.25 135.89 0)
+    (property "Value" "GND" (at 218.44 133.35 0)
       (effects (font (size 1.27 1.27)))
     )
@@
   )
   (symbol (lib_id "power:VBUS") (at 190.5 132.08 0) (unit 1)
-    (in_bom yes) (on_board yes) (dnp no) (fields_autoplaced)
+    (in_bom yes) (on_board yes) (dnp no)
     (property "Reference" "#PWR032" (at 190.5 135.89 0)
       (effects (font (size 1.27 1.27)) hide)
     )
-    (property "Value" "VBUS" (at 190.5 127 0)
+    (property "Value" "VBUS" (at 186.69 129.54 0)
       (effects (font (size 1.27 1.27)))
     )
@@
       (effects (font (size 1.27 1.27)) hide)
     )
-    (property "Value" "GND" (at 317.5 198.12 0)
+    (property "Value" "GND" (at 313.69 195.58 0)
       (effects (font (size 1.27 1.27)))
     )
@@
   )
   (symbol (lib_id "power:GND") (at 190.5 172.72 0) (unit 1)
-    (in_bom yes) (on_board yes) (dnp no) (fields_autoplaced)
+    (in_bom yes) (on_board yes) (dnp no)
     (property "Reference" "#PWR011" (at 190.5 179.07 0)
       (effects (font (size 1.27 1.27)) hide)
     )
-    (property "Value" "GND" (at 190.5 177.8 0)
-      (effects (font (size 1.27 1.27)))
-    )
+    (property "Value" "GND" (at 186.69 175.26 0)
+      (effects (font (size 1.27 1.27)))
+    )

Commit message: shrink MiniNDP
Parts:
- R1: renamed from R2; value 240k -> 200k
Other:
- note added: "(or AS6C4008)"
- note added: "AS6C2008A is optimal AS6C4008 is also compatible With AS6C4008 installed: Pin 6 is A17, high at all times, essentially inert, pin 9 is A18, receiving/returning the A17 data, resulting in the same outward functionality."
- note added: "Each ~{BLOCK} pulse resets A0-A9 to 0, and sets A10-A17 from BUS AD0-AD7. (0-255) Each ~{BYTE} pulse increments A0-A9 by 1. (0-1023)"
- note removed: "(AS6C4008)"
- note removed: "AS6C2008A (256Kx8) or AS6C4008 (512Kx8)"
- note removed: "AS6C2008A is optimal, but AS6C4008 is also compatible. With AS6C4008 installed: Pin 6 is A17, high at all times, essentially inert, pin 9 is A18, receiving/returning the A17 data, resulting in the same outward functionality."
- note removed: "Each ~{BLOCK} pulse updates local A10-A17 from BUS AD0-AD7 and resets the byte counter to 0. Each ~{BYTE} pulse disables SRAM, advances the byte counter by 1, and sets local A0-A9. 8 bits from the bus = 256 possible block-start addresses from the bus. 10 bits byte counter = 1k per block."
- note removed: "SYSTEM BUS connection is using STANDARD pin numbering for the connector, NOT the odd<>even swapped numbering from the TANDY Model 102 & 200 manuals. Example, RAM_RST is actually on pin 38, but the TANDY 102 & 200 manuals call it pin 37."
- moved on the sheet: BT1, C1, C2, C3, C4, C5, C6, D1, D2, J1, R1, U1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
