File: PCB/MiniNDP_512K_B.kicad_pcb (KiCad board)
At the start: 2 copper layers, 60 x 34 mm, 22 parts, among them J1 Conn_02x20_Odd_Even, U1 HC161, U2 HC161, U3 HC161, U4 HC138, U5 FCT821, U6 AS6C4008, U7 1G32

Commit message: new 512K_B board
Routing:
- net /A14: track 19.4 -> 20.3 mm
- net /A12: track 19.4 -> 20.3 mm
- net /A10: track 19.4 -> 20.3 mm
