File: PCB/MiniNDP_1M_B.kicad_pcb (KiCad board)
At the start: 2 copper layers, 60 x 34 mm, 22 parts, among them J1 Conn_02x20_Odd_Even, U1 HC161, U2 HC161, U3 HC161, U4 HC138, U5 FCT821, U6 AS6C8008_TSOPII, U7 1G32

Commit message: polish 512_B & 1M_B
Routing:
- net /~{WR}: track 34.0 -> 32.2 mm
- net /~{CE}: track 30.8 -> 29.1 mm
- net /AD2: track 32.8 -> 31.6 mm
- net /AD7: track 38.5 -> 37.7 mm
- net VBUS: track 113.4 -> 112.6 mm
- net /AD4: track 35.5 -> 34.7 mm
- net /AD3: track 29.8 -> 29.3 mm
- net /AD6: track 40.3 -> 40.8 mm
- net GND: vias 29 -> 33
Other:
- board text added: "BATTERY CR2032"
- board text added: "Use ENIG copper finish for gold plated battery terminal"

Commit message: 1M_B & 512_B
Parts:
- moved U7 1.30 mm to (149.9, 108.4)
- moved R2 1.30 mm to (154.4, 108.4)
- moved R3 1.30 mm to (152.3, 108.4)
- moved DA1 1.05 mm to (156.9, 108.5), turned to 90 degrees
Connections:
- net /BATT+ renamed +BATT
- net /~{CE} renamed /~{CE1}
Routing:
- net VMEM: track 40.2 -> 42.4 mm
- net /SLEEP: track 7.62 -> 9.59 mm
- net /~{CE1}: track 29.1 -> 30.4 mm
- net /~{BYTE}: track 46.2 -> 47.5 mm
- net /RAMRST: track 21.0 -> 19.7 mm
- net +BATT: track 43.7 -> 42.7 mm
- net /~{WR}: track 32.2 -> 33.2 mm
- net VBUS: track 112.6 -> 111.9 mm
