File: PCB/MiniNDP_OG.kicad_sch (KiCad schematic)
At the start: 20 parts, among them J1 Conn_02x20_Odd_Even, U1 HC161, U2 HC161, U3 HC161, U4 HC138, U5 HC574, U6 AS6C4008, U7 1G32, U8 1G79

Commit message: embed code font in pcb, bom export filename variables, delete extra battery trace
Other:
- title: MiniNDP -> MiniNDP_OG
