File: PCB/MiniNDP_OG.kicad_sch (KiCad schematic)
At the start: 20 parts, among them J1 Conn_02x20_Odd_Even, U1 HC161, U2 HC161, U3 HC161, U4 HC138, U5 HC574, U6 AS6C4008, U7 1G32, U8 1G79

Commit message: battery holder footprints
Parts:
- BT1: footprint 000_LOCAL:Keystone_3028_3034 -> 000_LOCAL:Keystone_3028_3034_bkw
Changed lines of the file:
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@@
 		)
 		(instances
-			(project "MiniNDP_512"
+			(project "MiniNDP_OG"
 				(path "/f15c2929-5cf4-4b4e-965d-148e1bec8a42"
 					(reference "C1")
@@
 		)
 		(instances
-			(project "MiniNDP_512"
+			(project "MiniNDP_OG"
 				(path "/f15c2929-5cf4-4b4e-965d-148e1bec8a42"
 					(reference "#PWR034")
@@
 		)
 		(instances
-			(project ""
+			(project "MiniNDP_OG"
 				(path "/f15c2929-5cf4-4b4e-965d-148e1bec8a42"
 					(reference "N1")
@@
 		)
 		(instances
-			(project "MiniNDP_512"
+			(project "MiniNDP_OG"
 				(path "/f15c2929-5cf4-4b4e-965d-148e1bec8a42"
 					(reference "U6")
@@
 		)
 		(instances
-			(project "MiniNDP_512_E"
+			(project "MiniNDP_OG"
 				(path "/f15c2929-5cf4-4b4e-965d-148e1bec8a42"
 					(reference "C5")
@@
 		)
 		(instances
-			(project "MiniNDP_512"
+			(project "MiniNDP_OG"
 				(path "/f15c2929-5cf4-4b4e-965d-148e1bec8a42"
 					(reference "#PWR08")
@@
 		)
 		(instances
-			(project "MiniNDP_512"
+			(project "MiniNDP_OG"
 				(path "/f15c2929-5cf4-4b4e-965d-148e1bec8a42"
 					(reference "#PWR010")
@@
 		)
 		(instances
-			(project "MiniNDP_512"
+			(project "MiniNDP_OG"
 				(path "/f15c2929-5cf4-4b4e-965d-148e1bec8a42"
 					(reference "#PWR01")
@@
 		)
 		(instances
-			(project "MiniNDP_512"
+			(project "MiniNDP_OG"
 				(path "/f15c2929-5cf4-4b4e-965d-148e1bec8a42"
 					(reference "JP1")
@@
 			)
 		)
-		(property "Footprint" "000_LOCAL:Keystone_3028_3034"
+		(property "Footprint" "000_LOCAL:Keystone_3028_3034_bkw"
 			(at 102.87 183.896 90)
 			(effects
@@
 		)
 		(instances
-			(project "MiniNDP_512"
+			(project "MiniNDP_OG"
 				(path "/f15c2929-5cf4-4b4e-965d-148e1bec8a42"
 					(reference "BT1")
@@
 		)
 		(instances
-			(project "MiniNDP_512"
+			(project "MiniNDP_OG"
 				(path "/f15c2929-5cf4-4b4e-965d-148e1bec8a42"
 					(reference "#PWR014")
@@
 		)
 		(instances
-			(project "MiniNDP_512"
+			(project "MiniNDP_OG"
 				(path "/f15c2929-5cf4-4b4e-965d-148e1bec8a42"
 					(reference "#PWR022")
@@
 		)
 		(instances
-			(project "MiniNDP_512"
+			(project "MiniNDP_OG"
 				(path "/f15c2929-5cf4-4b4e-965d-148e1bec8a42"
 					(reference "#PWR05")
@@
 		)
 		(instances
-			(project "MiniNDP_512"
+			(project "MiniNDP_OG"
 				(path "/f15c2929-5cf4-4b4e-965d-148e1bec8a42"
 					(reference "#PWR012")
@@
 		)
 		(instances
-			(project "MiniNDP_512"
+			(project "MiniNDP_OG"
 				(path "/f15c2929-5cf4-4b4e-965d-148e1bec8a42"
 					(reference "#FLG01")
@@
 		)
 		(instances
-			(project ""
+			(project "MiniNDP_OG"
 				(path "/f15c2929-5cf4-4b4e-965d-148e1bec8a42"
 					(reference "DA1")
@@
 		)
 		(instances
-			(project "MiniNDP_512"
+			(project "MiniNDP_OG"
 				(path "/f15c2929-5cf4-4b4e-965d-148e1bec8a42"
 					(reference "#PWR058")
@@
 		)
 		(instances
-			(project "MiniNDP_512"
+			(project "MiniNDP_OG"
 				(path "/f15c2929-5cf4-4b4e-965d-148e1bec8a42"
 					(reference "#PWR019")
@@
 		)
 		(instances
-			(project "MiniNDP_512"
+			(project "MiniNDP_OG"
 				(path "/f15c2929-5cf4-4b4e-965d-148e1bec8a42"
 					(reference "U3")
@@
 		)
 		(instances
-			(project "MiniNDP_512"
+			(project "MiniNDP_OG"
 				(path "/f15c2929-5cf4-4b4e-965d-148e1bec8a42"
 					(reference "#PWR07")
@@
 		)
 		(instances
-			(project "MiniNDP_512"
+			(project "MiniNDP_OG"
 				(path "/f15c2929-5cf4-4b4e-965d-148e1bec8a42"
 					(reference "#PWR042")
@@
 		)
 		(instances
-			(project "MiniNDP_512"
+			(project "MiniNDP_OG"
 				(path "/f15c2929-5cf4-4b4e-965d-148e1bec8a42"
 					(reference "#PWR057")
@@
 		)
 		(instances
-			(project ""
+			(project "MiniNDP_OG"
 				(path "/f15c2929-5cf4-4b4e-965d-148e1bec8a42"
 					(reference "U5")
@@
 		)
 		(instances
-			(project "MiniNDP_512"
+			(project "MiniNDP_OG"
 				(path "/f15c2929-5cf4-4b4e-965d-148e1bec8a42"
 					(reference "#PWR03")
@@
 		)
 		(instances
-			(project "MiniNDP_512"
+			(project "MiniNDP_OG"
 				(path "/f15c2929-5cf4-4b4e-965d-148e1bec8a42"
 					(reference "U1")
@@
 		)
 		(instances
-			(project "MiniNDP_512"
+			(project "MiniNDP_OG"
 				(path "/f15c2929-5cf4-4b4e-965d-148e1bec8a42"
 					(reference "#PWR055")
@@
 		)
 		(instances
-			(project "MiniNDP_512"
+			(project "MiniNDP_OG"
 				(path "/f15c2929-5cf4-4b4e-965d-148e1bec8a42"
 					(reference "U4")
@@
 		)
 		(instances
-			(project "MiniNDP_512"
+			(project "MiniNDP_OG"
 				(path "/f15c2929-5cf4-4b4e-965d-148e1bec8a42"
 					(reference "#PWR039")
@@
 		)
 		(instances
-			(project "MiniNDP_512"
+			(project "MiniNDP_OG"
 				(path "/f15c2929-5cf4-4b4e-965d-148e1bec8a42"
 					(reference "U7")
@@
 		)
 		(instances
-			(project "MiniNDP_512"
+			(project "MiniNDP_OG"
 				(path "/f15c2929-5cf4-4b4e-965d-148e1bec8a42"
 					(reference "#FLG03")
@@
 		)
 		(instances
-			(project "MiniNDP_512"
+			(project "MiniNDP_OG"
 				(path "/f15c2929-5cf4-4b4e-965d-148e1bec8a42"
 					(reference "#PWR023")
@@
 		)
 		(instances
-			(project "MiniNDP_512"
+			(project "MiniNDP_OG"
 				(path "/f15c2929-5cf4-4b4e-965d-148e1bec8a42"
 					(reference "U2")
@@
 		)
 		(instances
-			(project "MiniNDP_512"
+			(project "MiniNDP_OG"
 				(path "/f15c2929-5cf4-4b4e-965d-148e1bec8a42"
 					(reference "U8")
@@
 		)
 		(instances
-			(project "MiniNDP_512"
+			(project "MiniNDP_OG"
 				(path "/f15c2929-5cf4-4b4e-965d-148e1bec8a42"
 					(reference "#PWR06")
@@
 		)
 		(instances
-			(project "MiniNDP_512"
+			(project "MiniNDP_OG"
 				(path "/f15c2929-5cf4-4b4e-965d-148e1bec8a42"
 					(reference "#PWR038")
@@
 		)
 		(instances
-			(project "MiniNDP_512_E"
+			(project "MiniNDP_OG"
 				(path "/f15c2929-5cf4-4b4e-965d-148e1bec8a42"
 					(reference "C2")
@@
 		)
 		(instances
-			(project "MiniNDP_512"
+			(project "MiniNDP_OG"
 				(path "/f15c2929-5cf4-4b4e-965d-148e1bec8a42"
 					(reference "#PWR026")
@@
 		)
 		(instances
-			(project "MiniNDP_512"
+			(project "MiniNDP_OG"
 				(path "/f15c2929-5cf4-4b4e-965d-148e1bec8a42"
 					(reference "#PWR020")
@@
 		)
 		(instances
-			(project "MiniNDP_512"
+			(project "MiniNDP_OG"
 				(path "/f15c2929-5cf4-4b4e-965d-148e1bec8a42"
 					(reference "R2")
@@
 		)
 		(instances
-			(project "MiniNDP_512"
+			(project "MiniNDP_OG"
 				(path "/f15c2929-5cf4-4b4e-965d-148e1bec8a42"
 					(reference "#PWR04")
@@
 		)
 		(instances
-			(project "MiniNDP_512"
+			(project "MiniNDP_OG"
 				(path "/f15c2929-5cf4-4b4e-965d-148e1bec8a42"
 					(reference "#FLG02")
@@
 		)
 		(instances
-			(project "MiniNDP_512"
+			(project "MiniNDP_OG"
 				(path "/f15c2929-5cf4-4b4e-965d-148e1bec8a42"
 					(reference "#PWR09")
@@
 		)
 		(instances
-			(project "MiniNDP_512"
+			(project "MiniNDP_OG"
 				(path "/f15c2929-5cf4-4b4e-965d-148e1bec8a42"
 					(reference "#PWR015")
@@
 		)
 		(instances
-			(project "MiniNDP_512"
+			(project "MiniNDP_OG"
 				(path "/f15c2929-5cf4-4b4e-965d-148e1bec8a42"
 					(reference "#PWR021")
@@
 		)
 		(instances
-			(project "MiniNDP_512"
+			(project "MiniNDP_OG"
 				(path "/f15c2929-5cf4-4b4e-965d-148e1bec8a42"
 					(reference "#PWR02")
@@
 		)
 		(instances
-			(project "MiniNDP_512"
+			(project "MiniNDP_OG"
 				(path "/f15c2929-5cf4-4b4e-965d-148e1bec8a42"
 					(reference "#PWR025")
@@
 		)
 		(instances
-			(project "MiniNDP_512"
+			(project "MiniNDP_OG"
 				(path "/f15c2929-5cf4-4b4e-965d-148e1bec8a42"
 					(reference "#PWR018")
@@
 		)
 		(instances
-			(project "MiniNDP_512"
+			(project "MiniNDP_OG"
 				(path "/f15c2929-5cf4-4b4e-965d-148e1bec8a42"
 					(reference "R1")
@@
 		)
 		(instances
-			(project "MiniNDP_512"
+			(project "MiniNDP_OG"
 				(path "/f15c2929-5cf4-4b4e-965d-148e1bec8a42"
 					(reference "J1")
@@
 		)
 		(instances
-			(project "MiniNDP_512"
+			(project "MiniNDP_OG"
 				(path "/f15c2929-5cf4-4b4e-965d-148e1bec8a42"
 					(reference "#PWR041")
@@
 		)
 		(instances
-			(project "MiniNDP_512"
+			(project "MiniNDP_OG"
 				(path "/f15c2929-5cf4-4b4e-965d-148e1bec8a42"
 					(reference "#PWR032")
@@
 		)
 		(instances
-			(project "MiniNDP_512_E"
+			(project "MiniNDP_OG"
 				(path "/f15c2929-5cf4-4b4e-965d-148e1bec8a42"
 					(reference "C4")
@@
 		)
 		(instances
-			(project "MiniNDP_512"
+			(project "MiniNDP_OG"
 				(path "/f15c2929-5cf4-4b4e-965d-148e1bec8a42"
 					(reference "#PWR028")
@@
 		)
 		(instances
-			(project "MiniNDP_512"
+			(project "MiniNDP_OG"
 				(path "/f15c2929-5cf4-4b4e-965d-148e1bec8a42"
 					(reference "#PWR027")
@@
 		)
 		(instances
-			(project "MiniNDP_512"
+			(project "MiniNDP_OG"
 				(path "/f15c2929-5cf4-4b4e-965d-148e1bec8a42"
 					(reference "#PWR033")
@@
 		)
 		(instances
-			(project "MiniNDP_512_E"
+			(project "MiniNDP_OG"
 				(path "/f15c2929-5cf4-4b4e-965d-148e1bec8a42"
 					(reference "C3")
@@
 		)
 		(instances
-			(project "MiniNDP_512"
+			(project "MiniNDP_OG"
 				(path "/f15c2929-5cf4-4b4e-965d-148e1bec8a42"
 					(reference "#PWR017")
@@
 		)
 		(instances
-			(project "MiniNDP_512"
+			(project "MiniNDP_OG"
 				(path "/f15c2929-5cf4-4b4e-965d-148e1bec8a42"
 					(reference "#PWR011")
@@
 		)
 		(instances
-			(project "MiniNDP_512"
+			(project "MiniNDP_OG"
 				(path "/f15c2929-5cf4-4b4e-965d-148e1bec8a42"
 					(reference "#PWR016")
