File: PCB/MiniNDP_SL1M.kicad_sch (KiCad schematic)
At the start: 14 parts, among them J1 Conn_02x20_Odd_Even, U1 AS6C8008_TSOPII, U2 HC238, U3 HC4040, U4 ABT841

Commit message: embed code font in pcb, bom export filename variables, delete extra battery trace
Other:
- title: MiniNDP -> MiniNDP_SL1M
