File: PCB/MiniNDP_SL1M.kicad_sch (KiCad schematic)
At the start: 14 parts, among them J1 Conn_02x20_Odd_Even, U1 AS6C8008_TSOPII, U2 HC238, U3 HC4040, U4 ABT841

Commit message: fix tssop-24 model, update cover models
Parts:
- U4: footprint 000_LOCAL:TSSOP-24_4.4x7.8mm_P0.65mm -> 000_LOCAL:TSSOP-24
Changed lines of the file:
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@@
 		)
 		(instances
-			(project "MiniNDP_1M_B"
+			(project "MiniNDP_SL1M"
 				(path "/f15c2929-5cf4-4b4e-965d-148e1bec8a42"
 					(reference "U1")
@@
 		)
 		(instances
-			(project "MiniNDP_1M_B"
+			(project "MiniNDP_SL1M"
 				(path "/f15c2929-5cf4-4b4e-965d-148e1bec8a42"
 					(reference "#PWR08")
@@
 		)
 		(instances
-			(project ""
+			(project "MiniNDP_SL1M"
 				(path "/f15c2929-5cf4-4b4e-965d-148e1bec8a42"
 					(reference "U2")
@@
 		)
 		(instances
-			(project "MiniNDP_1M_B"
+			(project "MiniNDP_SL1M"
 				(path "/f15c2929-5cf4-4b4e-965d-148e1bec8a42"
 					(reference "#PWR010")
@@
 		)
 		(instances
-			(project "MiniNDP_1M_B"
+			(project "MiniNDP_SL1M"
 				(path "/f15c2929-5cf4-4b4e-965d-148e1bec8a42"
 					(reference "#PWR01")
@@
 		)
 		(instances
-			(project "MiniNDP_1M_B"
+			(project "MiniNDP_SL1M"
 				(path "/f15c2929-5cf4-4b4e-965d-148e1bec8a42"
 					(reference "BT1")
@@
 		)
 		(instances
-			(project "MiniNDP_1M_B"
+			(project "MiniNDP_SL1M"
 				(path "/f15c2929-5cf4-4b4e-965d-148e1bec8a42"
 					(reference "#PWR022")
@@
 		)
 		(instances
-			(project "MiniNDP_1M_B"
+			(project "MiniNDP_SL1M"
 				(path "/f15c2929-5cf4-4b4e-965d-148e1bec8a42"
 					(reference "#PWR05")
@@
 		)
 		(instances
-			(project "MiniNDP_1M_B"
+			(project "MiniNDP_SL1M"
 				(path "/f15c2929-5cf4-4b4e-965d-148e1bec8a42"
 					(reference "#PWR012")
@@
 		)
 		(instances
-			(project "MiniNDP_1M_B"
+			(project "MiniNDP_SL1M"
 				(path "/f15c2929-5cf4-4b4e-965d-148e1bec8a42"
 					(reference "#FLG01")
@@
 		)
 		(instances
-			(project "MiniNDP_1M_B"
+			(project "MiniNDP_SL1M"
 				(path "/f15c2929-5cf4-4b4e-965d-148e1bec8a42"
 					(reference "#PWR058")
@@
 		)
 		(instances
-			(project "MiniNDP_1M_B"
+			(project "MiniNDP_SL1M"
 				(path "/f15c2929-5cf4-4b4e-965d-148e1bec8a42"
 					(reference "#PWR019")
@@
 		)
 		(instances
-			(project "MiniNDP_1M_B"
+			(project "MiniNDP_SL1M"
 				(path "/f15c2929-5cf4-4b4e-965d-148e1bec8a42"
 					(reference "#PWR07")
@@
 		)
 		(instances
-			(project "MiniNDP_1M_B"
+			(project "MiniNDP_SL1M"
 				(path "/f15c2929-5cf4-4b4e-965d-148e1bec8a42"
 					(reference "#PWR042")
@@
 		)
 		(instances
-			(project "MiniNDP_1M_B"
+			(project "MiniNDP_SL1M"
 				(path "/f15c2929-5cf4-4b4e-965d-148e1bec8a42"
 					(reference "#PWR057")
@@
 		)
 		(instances
-			(project "MiniNDP_1M_B"
+			(project "MiniNDP_SL1M"
 				(path "/f15c2929-5cf4-4b4e-965d-148e1bec8a42"
 					(reference "#PWR03")
@@
 		)
 		(instances
-			(project "MiniNDP_1M_B"
+			(project "MiniNDP_SL1M"
 				(path "/f15c2929-5cf4-4b4e-965d-148e1bec8a42"
 					(reference "#PWR055")
@@
 		)
 		(instances
-			(project "MiniNDP_1M_F_thin"
+			(project "MiniNDP_SL1M"
 				(path "/f15c2929-5cf4-4b4e-965d-148e1bec8a42"
 					(reference "DA1")
@@
 		)
 		(instances
-			(project "MiniNDP_1M"
+			(project "MiniNDP_SL1M"
 				(path "/f15c2929-5cf4-4b4e-965d-148e1bec8a42"
 					(reference "N1")
@@
 		)
 		(instances
-			(project "MiniNDP_1M_F_thin"
+			(project "MiniNDP_SL1M"
 				(path "/f15c2929-5cf4-4b4e-965d-148e1bec8a42"
 					(reference "C5")
@@
 		)
 		(instances
-			(project "MiniNDP_1M_C"
+			(project "MiniNDP_SL1M"
 				(path "/f15c2929-5cf4-4b4e-965d-148e1bec8a42"
 					(reference "C2")
@@
 		)
 		(instances
-			(project "MiniNDP_1M_B"
+			(project "MiniNDP_SL1M"
 				(path "/f15c2929-5cf4-4b4e-965d-148e1bec8a42"
 					(reference "#FLG03")
@@
 		)
 		(instances
-			(project "MiniNDP_1M_B"
+			(project "MiniNDP_SL1M"
 				(path "/f15c2929-5cf4-4b4e-965d-148e1bec8a42"
 					(reference "#PWR023")
@@
 		)
 		(instances
-			(project "MiniNDP_1M_B"
+			(project "MiniNDP_SL1M"
 				(path "/f15c2929-5cf4-4b4e-965d-148e1bec8a42"
 					(reference "#PWR06")
@@
 		)
 		(instances
-			(project ""
+			(project "MiniNDP_SL1M"
 				(path "/f15c2929-5cf4-4b4e-965d-148e1bec8a42"
 					(reference "U3")
@@
 		)
 		(instances
-			(project "MiniNDP_1M_B"
+			(project "MiniNDP_SL1M"
 				(path "/f15c2929-5cf4-4b4e-965d-148e1bec8a42"
 					(reference "#PWR027")
@@
 		)
 		(instances
-			(project "MiniNDP_1M"
+			(project "MiniNDP_SL1M"
 				(path "/f15c2929-5cf4-4b4e-965d-148e1bec8a42"
 					(reference "#PWR014")
@@
 		)
 		(instances
-			(project "MiniNDP_1M_B"
+			(project "MiniNDP_SL1M"
 				(path "/f15c2929-5cf4-4b4e-965d-148e1bec8a42"
 					(reference "R1")
@@
 		)
 		(instances
-			(project "MiniNDP_1M_B"
+			(project "MiniNDP_SL1M"
 				(path "/f15c2929-5cf4-4b4e-965d-148e1bec8a42"
 					(reference "#PWR04")
@@
 		)
 		(instances
-			(project "MiniNDP_1M_B"
+			(project "MiniNDP_SL1M"
 				(path "/f15c2929-5cf4-4b4e-965d-148e1bec8a42"
 					(reference "#FLG02")
@@
 		)
 		(instances
-			(project "MiniNDP_1M_B"
+			(project "MiniNDP_SL1M"
 				(path "/f15c2929-5cf4-4b4e-965d-148e1bec8a42"
 					(reference "#PWR09")
@@
 		)
 		(instances
-			(project "MiniNDP_1M_C06"
+			(project "MiniNDP_SL1M"
 				(path "/f15c2929-5cf4-4b4e-965d-148e1bec8a42"
 					(reference "C4")
@@
 		)
 		(instances
-			(project "MiniNDP_1M_B"
+			(project "MiniNDP_SL1M"
 				(path "/f15c2929-5cf4-4b4e-965d-148e1bec8a42"
 					(reference "#PWR025")
@@
 		)
 		(instances
-			(project "MiniNDP_1M_B"
+			(project "MiniNDP_SL1M"
 				(path "/f15c2929-5cf4-4b4e-965d-148e1bec8a42"
 					(reference "J1")
@@
 		)
 		(instances
-			(project "MiniNDP_1M_B"
+			(project "MiniNDP_SL1M"
 				(path "/f15c2929-5cf4-4b4e-965d-148e1bec8a42"
 					(reference "#PWR041")
@@
 		)
 		(instances
-			(project "MiniNDP_1M_C"
+			(project "MiniNDP_SL1M"
 				(path "/f15c2929-5cf4-4b4e-965d-148e1bec8a42"
 					(reference "C3")
@@
 		)
 		(instances
-			(project "MiniNDP_1M_B"
+			(project "MiniNDP_SL1M"
 				(path "/f15c2929-5cf4-4b4e-965d-148e1bec8a42"
 					(reference "#PWR032")
@@
 			)
 		)
-		(property "Footprint" "000_LOCAL:TSSOP-24_4.4x7.8mm_P0.65mm"
+		(property "Footprint" "000_LOCAL:TSSOP-24"
 			(at 152.4 104.14 0)
 			(effects
@@
 		)
 		(instances
-			(project ""
+			(project "MiniNDP_SL1M"
 				(path "/f15c2929-5cf4-4b4e-965d-148e1bec8a42"
 					(reference "U4")
@@
 		)
 		(instances
-			(project "MiniNDP_1M_B"
+			(project "MiniNDP_SL1M"
 				(path "/f15c2929-5cf4-4b4e-965d-148e1bec8a42"
 					(reference "#PWR033")
@@
 		)
 		(instances
-			(project "MiniNDP_1M_B"
+			(project "MiniNDP_SL1M"
 				(path "/f15c2929-5cf4-4b4e-965d-148e1bec8a42"
 					(reference "#PWR011")
@@
 		)
 		(instances
-			(project "MiniNDP_1M_B"
+			(project "MiniNDP_SL1M"
 				(path "/f15c2929-5cf4-4b4e-965d-148e1bec8a42"
 					(reference "C1")
@@
 		)
 		(instances
-			(project "MiniNDP_1M_B"
+			(project "MiniNDP_SL1M"
 				(path "/f15c2929-5cf4-4b4e-965d-148e1bec8a42"
 					(reference "#PWR016")

Commit message: add sram part numbers to 1M versions sch
Other:
- note added: "AS6C8008-xxZ CY62158ELL"
Changed lines of the file:
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@@
+		)
+	)
+	(text "AS6C8008-xxZ\nCY62158ELL"
+		(exclude_from_sim no)
+		(at 228.6 25.4 0)
+		(effects
+			(font
+				(size 1.27 1.27)
+			)
 		)
 	)

Commit message: simplify covers, strengthen battery holders, silkscreen, readme
Parts:
- BT1: footprint 000_LOCAL:Keystone_3028_3034 -> 000_LOCAL:Keystone_3028_3034_bkw
Other:
- moved on the sheet: U2, U3
