File: PCB/MiniNDP_u1M.kicad_pcb (KiCad board)
At the start: 2 copper layers, 51.3 x 18.3 mm, 15 parts, among them J1 Model_100_System_BUS, U1 AS6C8008_TSOPII, U2 HC238, U3 HC4040, U4 ABT841

Commit message: u1M 023 trivial pcb polish
Routing:
- net VMEM: track 37.9 -> 39.3 mm
- net GND: vias 56 -> 57
