File: PCB/MiniNDP_512_Breadboard.kicad_sch (KiCad schematic)
At the start: 9 parts, among them J1 Conn_02x20_Odd_Even, U1 HC161, U2 HC161, U3 HC161, U4 HC138, U5 HC374, U6 AS6C4008, U7 HC32, U8 HC374

Commit message: rename breadboard, sl1m trace spacing & silkscreen
Other:
- title: MiniNDP 512 DIP Breadboard -> MiniNDP 512 Breadboard
