File: PCB/MiniNDP_EZ256.kicad_pcb (KiCad board)
At the start: 2 copper layers, 60 x 34 mm, 22 parts, among them J1 Conn_02x20_Odd_Even, U1 HC238, U2 HC4040, U3 HC573, U4 AS6C2008A

Commit message: ez256 compatible with 128k sram
Connections:
- U3 pad 7: /AD7 -> /AD3
- U3 pad 8: /AD3 -> /AD4
- U3 pad 9: /AD4 -> /AD7
- U4 pad 1: /A9 -> /A17
- U4 pad 2: /A7 -> /A9
- U4 pad 28: /A8 -> /A7
- U4 pad 3: /A17 -> /A8
Routing:
- net /A7: track 27.9 -> 13.5 mm
- net /A8: track 14.6 -> 28.0 mm
- net /A17: track 16.4 -> 21.0 mm
- net /AD4: track 42.9 -> 40.7 mm
- net /AD3: track 41.1 -> 39.0 mm
- net /RAMRST: track 52.4 -> 50.3 mm
- net /AD7: track 31.6 -> 29.8 mm, vias 1 -> 2
- net /A9: track 27.9 -> 26.4 mm
- net /A2: track 18.1 -> 17.0 mm
- net /~{RD}: track 32.6 -> 31.6 mm
- net /A1: track 17.9 -> 17.0 mm
- net /(A): track 44.1 -> 43.4 mm
- net /AD2: track 44.3 -> 44.8 mm
- net /~{WR}: track 28.0 -> 27.5 mm
- net GND: vias 61 -> 74
Other:
- board text added: "128k 256k"
- board text added: "BASIC to bootstrap RAMxxx.CO previously saved as the first file on the device"
- board text removed: "Bootstrap install RAMDSK from the card. RAM100.CO or RAM200.CO must be the first file on the card."

Commit message: M10 & EZ256 trace & via clearances, silkscreen
Connections:
- J1 pad 16: /BUS_A10 -> unconnected-(J1-Pin_16-Pad16)
Routing:
- net /A11: track 21.3 -> 18.5 mm
- net /A10: track 20.5 -> 18.1 mm
- net /A12: track 19.9 -> 18.7 mm
- net /A13: track 18.5 -> 17.6 mm
- net /A14: track 17.5 -> 16.9 mm
- net VBUS: track 128.3 -> 128.8 mm
- net GND: vias 74 -> 77
