File: PCB/MiniNDP_M10x.kicad_sch (KiCad schematic)
At the start: 14 parts, among them J1 Conn_02x20_Odd_Even, U1 AS6C8008_TSOPII, U2 HC238, U3 HC4040, U4 ABT841

Commit message: M10x M-10 w/std pcb outline & std thin cover
Parts:
- N1: value MiniNDP_Cover_M10 -> MiniNDP_Cover_THIN
Connections:
- net AD0: now also U1.35 (Q6), U4.5 (D3); no longer U1.32 (Q5), U4.10 (D8)
- net AD1: now also U1.36 (Q7), U4.4 (D2); no longer U1.31 (Q4), U4.11 (D9)
- net AD2: now also U1.10 (Q1), U4.7 (D5); no longer U1.35 (Q6), U4.5 (D3)
- net AD3: now also U1.9 (Q0), U4.6 (D4); no longer U1.36 (Q7), U4.4 (D2)
- net AD4: now also U1.14 (Q3), U4.9 (D7); no longer U1.10 (Q1), U4.7 (D5)
- net AD5: now also U1.13 (Q2), U4.8 (D6); no longer U1.9 (Q0), U4.6 (D4)
- net AD6: now also U1.31 (Q4), U4.11 (D9); no longer U1.14 (Q3), U4.9 (D7)
- net AD7: now also U1.32 (Q5), U4.10 (D8); no longer U1.13 (Q2), U4.8 (D6)
- net BUS_A10: now also U4.3 (D1); no longer U4.2 (D0)
- net BUS_A11: now also U4.2 (D0); no longer U4.3 (D1)
Other:
- note added: "CR2012 battery holder and THIN cover just barely allows access to the M-10 batteries without removing the card."
- title: MiniNDP_M10 -> MiniNDP
Changed lines of the file:
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@@
 	(paper "A4")
 	(title_block
-		(title "MiniNDP_M10")
-		(date "2026-07-23")
-		(rev "01")
+		(title "MiniNDP")
+		(date "2026-08-09")
+		(rev "M10x_01")
 		(company "Brian K. White - b.kenyon.w@gmail.com")
 		(comment 1 "github.com/bkw777/NODE_DATAPAC")
@@
 		)
 	)
+	(text "CR2012 battery holder and THIN cover\njust barely allows access to the M-10\nbatteries without removing the card."
+		(exclude_from_sim no)
+		(at 37.084 158.75 0)
+		(effects
+			(font
+				(size 1.27 1.27)
+			)
+			(justify left)
+		)
+	)
 	(text "		BUS  BUS  BUS  BUS\n(A)	~{YO}   _A8  _A9  _A10  _A11  ->  ~{BLOCK} ~{BYTE}\n L	 X	 X	  X	  X	   X		X	  X\n X	 H	 X	  X	  X	   X		X	  X\n X	 X	 L	  X	  X	   X		X	  X\n H	 L	 H	  L	  L	   L	->  H	  L  Select BLOCK N, BANK0: OUT129,N\n H	 L	 H	  L	  H	   L	->  H	  L  Select BLOCK N, BANK1: OUT133,N\n H	 L	 H	  L	  L	   H	->  H	  L  Select BLOCK N, BANK2: OUT137,N\n H	 L	 H	  L	  H	   H	->  H	  L  Select BLOCK N, BANK3: OUT141,N\n H	 L	 H	  H	  X	   X	->  L	  H  READ N: N=INP(131) or WRITE N: OUT131,N\n\nBLOCK\nH: sets A0-A9 to 0, updates A10-A19 from AD0-AD7 & BUS_A10-BUS_A11\nL: latches A10-A19\n\nBYTE\nH: enables SRAM for read or write\nL: disables SRAM, increments A0-A9 by 1\n"
 		(exclude_from_sim no)
@@
 	)
 	(label "BUS_A11"
-		(at 139.7 93.98 180)
+		(at 139.7 91.44 180)
 		(effects
 			(font
@@
 	)
 	(label "AD5"
-		(at 139.7 101.6 180)
+		(at 139.7 106.68 180)
 		(effects
 			(font
@@
 	)
 	(label "AD0"
-		(at 241.3 53.34 0)
+		(at 241.3 55.88 0)
 		(effects
 			(font
@@
 	)
 	(label "AD6"
-		(at 139.7 109.22 180)
+		(at 139.7 114.3 180)
 		(effects
 			(font
@@
 	)
 	(label "AD5"
-		(at 241.3 40.64 0)
+		(at 241.3 45.72 0)
 		(effects
 			(font
@@
 	)
 	(label "AD1"
-		(at 241.3 50.8 0)
+		(at 241.3 58.42 0)
 		(effects
 			(font
@@
 	)
 	(label "AD0"
-		(at 139.7 111.76 180)
+		(at 139.7 99.06 180)
 		(effects
 			(font
@@
 	)
 	(label "AD4"
-		(at 139.7 104.14 180)
+		(at 139.7 109.22 180)
 		(effects
 			(font
@@
 	)
 	(label "AD7"
-		(at 241.3 45.72 0)
+		(at 241.3 53.34 0)
 		(effects
 			(font
@@
 	)
 	(label "AD4"
-		(at 241.3 43.18 0)
+		(at 241.3 48.26 0)
 		(effects
 			(font
@@
 	)
 	(label "AD2"
-		(at 139.7 99.06 180)
+		(at 139.7 104.14 180)
 		(effects
 			(font
@@
 	)
 	(label "BUS_A10"
-		(at 139.7 91.44 180)
+		(at 139.7 93.98 180)
 		(effects
 			(font
@@
 	)
 	(label "AD3"
-		(at 241.3 58.42 0)
+		(at 241.3 40.64 0)
 		(effects
 			(font
@@
 	)
 	(label "AD2"
-		(at 241.3 55.88 0)
+		(at 241.3 43.18 0)
 		(effects
 			(font
@@
 	)
 	(label "AD7"
-		(at 139.7 106.68 180)
+		(at 139.7 111.76 180)
 		(effects
 			(font
@@
 	)
 	(label "AD1"
-		(at 139.7 114.3 180)
+		(at 139.7 96.52 180)
 		(effects
 			(font
@@
 	)
 	(label "AD6"
-		(at 241.3 48.26 0)
+		(at 241.3 50.8 0)
 		(effects
 			(font
@@
 	)
 	(label "AD3"
-		(at 139.7 96.52 180)
+		(at 139.7 101.6 180)
 		(effects
 			(font
@@
 		)
 		(instances
-			(project "MiniNDP_M10"
+			(project "MiniNDP_M10x"
 				(path "/f15c2929-5cf4-4b4e-965d-148e1bec8a42"
 					(reference "U1")
@@
 		)
 		(instances
-			(project "MiniNDP_M10"
+			(project "MiniNDP_M10x"
 				(path "/f15c2929-5cf4-4b4e-965d-148e1bec8a42"
 					(reference "#PWR08")
@@
 		)
 		(instances
-			(project "MiniNDP_M10"
+			(project "MiniNDP_M10x"
 				(path "/f15c2929-5cf4-4b4e-965d-148e1bec8a42"
 					(reference "U2")
@@
 		)
 		(instances
-			(project "MiniNDP_M10"
+			(project "MiniNDP_M10x"
 				(path "/f15c2929-5cf4-4b4e-965d-148e1bec8a42"
 					(reference "#PWR010")
@@
 		)
 		(instances
-			(project "MiniNDP_M10"
+			(project "MiniNDP_M10x"
 				(path "/f15c2929-5cf4-4b4e-965d-148e1bec8a42"
 					(reference "#PWR01")
@@
 		)
 		(instances
-			(project "MiniNDP_M10"
+			(project "MiniNDP_M10x"
 				(path "/f15c2929-5cf4-4b4e-965d-148e1bec8a42"
 					(reference "BT1")
@@
 		)
 		(instances
-			(project "MiniNDP_M10"
+			(project "MiniNDP_M10x"
 				(path "/f15c2929-5cf4-4b4e-965d-148e1bec8a42"
 					(reference "#PWR022")
@@
 		)
 		(instances
-			(project "MiniNDP_M10"
+			(project "MiniNDP_M10x"
 				(path "/f15c2929-5cf4-4b4e-965d-148e1bec8a42"
 					(reference "#PWR05")
@@
 		)
 		(instances
-			(project "MiniNDP_M10"
+			(project "MiniNDP_M10x"
 				(path "/f15c2929-5cf4-4b4e-965d-148e1bec8a42"
 					(reference "#PWR012")
@@
 		)
 		(instances
-			(project "MiniNDP_M10"
+			(project "MiniNDP_M10x"
 				(path "/f15c2929-5cf4-4b4e-965d-148e1bec8a42"
 					(reference "#FLG01")
@@
 		)
 		(instances
-			(project "MiniNDP_M10"
+			(project "MiniNDP_M10x"
 				(path "/f15c2929-5cf4-4b4e-965d-148e1bec8a42"
 					(reference "#PWR058")
@@
 		)
 		(instances
-			(project "MiniNDP_M10"
+			(project "MiniNDP_M10x"
 				(path "/f15c2929-5cf4-4b4e-965d-148e1bec8a42"
 					(reference "#PWR019")
@@
 		)
 		(instances
-			(project "MiniNDP_M10"
+			(project "MiniNDP_M10x"
 				(path "/f15c2929-5cf4-4b4e-965d-148e1bec8a42"
 					(reference "#PWR07")
@@
 		)
 		(instances
-			(project "MiniNDP_M10"
+			(project "MiniNDP_M10x"
 				(path "/f15c2929-5cf4-4b4e-965d-148e1bec8a42"
 					(reference "#PWR042")
@@
 		)
 		(instances
-			(project "MiniNDP_M10"
+			(project "MiniNDP_M10x"
 				(path "/f15c2929-5cf4-4b4e-965d-148e1bec8a42"
 					(reference "#PWR057")
@@
 		)
 		(instances
-			(project "MiniNDP_M10"
+			(project "MiniNDP_M10x"
 				(path "/f15c2929-5cf4-4b4e-965d-148e1bec8a42"
 					(reference "#PWR03")
@@
 		)
 		(instances
-			(project "MiniNDP_M10"
+			(project "MiniNDP_M10x"
 				(path "/f15c2929-5cf4-4b4e-965d-148e1bec8a42"
 					(reference "#PWR055")
@@
 		)
 		(instances
-			(project "MiniNDP_M10"
+			(project "MiniNDP_M10x"
 				(path "/f15c2929-5cf4-4b4e-965d-148e1bec8a42"
 					(reference "DA1")
@@
 			)
 		)
-		(property "Value" "MiniNDP_Cover_M10"
+		(property "Value" "MiniNDP_Cover_THIN"
 			(at 26.67 149.352 0)
 			(effects
@@
 		)
 		(instances
-			(project "MiniNDP_M10"
+			(project "MiniNDP_M10x"
 				(path "/f15c2929-5cf4-4b4e-965d-148e1bec8a42"
 					(reference "N1")
@@
 		)
 		(instances
-			(project "MiniNDP_M10"
+			(project "MiniNDP_M10x"
 				(path "/f15c2929-5cf4-4b4e-965d-148e1bec8a42"
 					(reference "C5")
@@
 		)
 		(instances
-			(project "MiniNDP_M10"
+			(project "MiniNDP_M10x"
 				(path "/f15c2929-5cf4-4b4e-965d-148e1bec8a42"
 					(reference "C2")
@@
 		)
 		(instances
-			(project "MiniNDP_M10"
+			(project "MiniNDP_M10x"
 				(path "/f15c2929-5cf4-4b4e-965d-148e1bec8a42"
 					(reference "#FLG03")
@@
 		)
 		(instances
-			(project "MiniNDP_M10"
+			(project "MiniNDP_M10x"
 				(path "/f15c2929-5cf4-4b4e-965d-148e1bec8a42"
 					(reference "#PWR023")
@@
 		)
 		(instances
-			(project "MiniNDP_M10"
+			(project "MiniNDP_M10x"
 				(path "/f15c2929-5cf4-4b4e-965d-148e1bec8a42"
 					(reference "#PWR06")
@@
 		)
 		(instances
-			(project "MiniNDP_M10"
+			(project "MiniNDP_M10x"
 				(path "/f15c2929-5cf4-4b4e-965d-148e1bec8a42"
 					(reference "U3")
@@
 		)
 		(instances
-			(project "MiniNDP_M10"
+			(project "MiniNDP_M10x"
 				(path "/f15c2929-5cf4-4b4e-965d-148e1bec8a42"
 					(reference "#PWR027")
@@
 		)
 		(instances
-			(project "MiniNDP_M10"
+			(project "MiniNDP_M10x"
 				(path "/f15c2929-5cf4-4b4e-965d-148e1bec8a42"
 					(reference "#PWR014")
@@
 		)
 		(instances
-			(project "MiniNDP_M10"
+			(project "MiniNDP_M10x"
 				(path "/f15c2929-5cf4-4b4e-965d-148e1bec8a42"
 					(reference "R1")
@@
 		)
 		(instances
-			(project "MiniNDP_M10"
+			(project "MiniNDP_M10x"
 				(path "/f15c2929-5cf4-4b4e-965d-148e1bec8a42"
 					(reference "#PWR04")
@@
 		)
 		(instances
-			(project "MiniNDP_M10"
+			(project "MiniNDP_M10x"
 				(path "/f15c2929-5cf4-4b4e-965d-148e1bec8a42"
 					(reference "#FLG02")
@@
 		)
 		(instances
-			(project "MiniNDP_M10"
+			(project "MiniNDP_M10x"
 				(path "/f15c2929-5cf4-4b4e-965d-148e1bec8a42"
 					(reference "#PWR09")
@@
 		)
 		(instances
-			(project "MiniNDP_M10"
+			(project "MiniNDP_M10x"
 				(path "/f15c2929-5cf4-4b4e-965d-148e1bec8a42"
 					(reference "C4")
@@
 		)
 		(instances
-			(project "MiniNDP_M10"
+			(project "MiniNDP_M10x"
 				(path "/f15c2929-5cf4-4b4e-965d-148e1bec8a42"
 					(reference "#PWR025")
@@
 		)
 		(instances
-			(project "MiniNDP_M10"
+			(project "MiniNDP_M10x"
 				(path "/f15c2929-5cf4-4b4e-965d-148e1bec8a42"
 					(reference "J1")
@@
 		)
 		(instances
-			(project "MiniNDP_M10"
+			(project "MiniNDP_M10x"
 				(path "/f15c2929-5cf4-4b4e-965d-148e1bec8a42"
 					(reference "#PWR041")
@@
 		)
 		(instances
-			(project "MiniNDP_M10"
+			(project "MiniNDP_M10x"
 				(path "/f15c2929-5cf4-4b4e-965d-148e1bec8a42"
 					(reference "C3")
@@
 		)
 		(instances
-			(project "MiniNDP_M10"
+			(project "MiniNDP_M10x"
 				(path "/f15c2929-5cf4-4b4e-965d-148e1bec8a42"
 					(reference "#PWR032")
@@
 		)
 		(instances
-			(project "MiniNDP_M10"
+			(project "MiniNDP_M10x"
 				(path "/f15c2929-5cf4-4b4e-965d-148e1bec8a42"
 					(reference "U4")
@@
 		)
 		(instances
-			(project "MiniNDP_M10"
+			(project "MiniNDP_M10x"
 				(path "/f15c2929-5cf4-4b4e-965d-148e1bec8a42"
 					(reference "#PWR033")
@@
 		)
 		(instances
-			(project "MiniNDP_M10"
+			(project "MiniNDP_M10x"
 				(path "/f15c2929-5cf4-4b4e-965d-148e1bec8a42"
 					(reference "#PWR011")
@@
 		)
 		(instances
-			(project "MiniNDP_M10"
+			(project "MiniNDP_M10x"
 				(path "/f15c2929-5cf4-4b4e-965d-148e1bec8a42"
 					(reference "C1")
@@
 		)
 		(instances
-			(project "MiniNDP_M10"
+			(project "MiniNDP_M10x"
 				(path "/f15c2929-5cf4-4b4e-965d-148e1bec8a42"
 					(reference "#PWR016")
