File: PCB/MiniNDP_M10x2.kicad_sch (KiCad schematic)
At the start: 14 parts, among them J1 Conn_02x20_Odd_Even, U1 AS6C8008_TSOPII, U2 HC238, U3 HC4040, U4 ABT841

Commit message: Olivetti M-10 take 3. T512 pics readme.
Parts:
- N1: value MiniNDP_Cover_M10 -> MiniNDP_Cover_M10compact2; footprint 000_LOCAL:MiniNDP_Cover_M10 -> 000_LOCAL:MiniNDP_Cover_M10compact2; MPN MiniNDP_Cover_M10.stl -> MiniNDP_Cover_M10compact2.stl
Other:
- note removed: "1M for Olivetti M-10"
- title: MiniNDP_M10 -> MiniNDP_M10c2
Changed lines of the file:
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@@
 	(paper "USLetter")
 	(title_block
-		(title "MiniNDP_M10")
+		(title "MiniNDP_M10c2")
 		(date "2026-08-13")
-		(rev "20")
+		(rev "01")
 		(company "Brian K. White - b.kenyon.w@gmail.com")
 		(comment 1 "github.com/bkw777/NODE_DATAPAC")
@@
 		)
 	)
-	(text "1M for Olivetti M-10"
-		(exclude_from_sim no)
-		(at 234.442 180.086 0)
-		(effects
-			(font
-				(size 2.54 2.54)
-			)
-		)
-	)
 	(text "VDD"
 		(exclude_from_sim no)
@@
 		)
 		(instances
-			(project "MiniNDP_M10"
+			(project "MiniNDP_M10x2"
 				(path "/28a4b045-d480-4410-adb7-fa6b33984079"
 					(reference "U1")
@@
 		)
 		(instances
-			(project "MiniNDP_M10"
+			(project "MiniNDP_M10x2"
 				(path "/28a4b045-d480-4410-adb7-fa6b33984079"
 					(reference "#PWR08")
@@
 		)
 		(instances
-			(project "MiniNDP_M10"
+			(project "MiniNDP_M10x2"
 				(path "/28a4b045-d480-4410-adb7-fa6b33984079"
 					(reference "U2")
@@
 		)
 		(instances
-			(project "MiniNDP_M10"
+			(project "MiniNDP_M10x2"
 				(path "/28a4b045-d480-4410-adb7-fa6b33984079"
 					(reference "#PWR010")
@@
 		)
 		(instances
-			(project "MiniNDP_M10"
+			(project "MiniNDP_M10x2"
 				(path "/28a4b045-d480-4410-adb7-fa6b33984079"
 					(reference "#PWR01")
@@
 		)
 		(instances
-			(project "MiniNDP_M10"
+			(project "MiniNDP_M10x2"
 				(path "/28a4b045-d480-4410-adb7-fa6b33984079"
 					(reference "BT1")
@@
 		)
 		(instances
-			(project "MiniNDP_M10"
+			(project "MiniNDP_M10x2"
 				(path "/28a4b045-d480-4410-adb7-fa6b33984079"
 					(reference "#PWR022")
@@
 		)
 		(instances
-			(project "MiniNDP_M10"
+			(project "MiniNDP_M10x2"
 				(path "/28a4b045-d480-4410-adb7-fa6b33984079"
 					(reference "#PWR05")
@@
 		)
 		(instances
-			(project "MiniNDP_M10"
+			(project "MiniNDP_M10x2"
 				(path "/28a4b045-d480-4410-adb7-fa6b33984079"
 					(reference "#PWR012")
@@
 		)
 		(instances
-			(project "MiniNDP_M10"
+			(project "MiniNDP_M10x2"
 				(path "/28a4b045-d480-4410-adb7-fa6b33984079"
 					(reference "#FLG01")
@@
 		)
 		(instances
-			(project "MiniNDP_M10"
+			(project "MiniNDP_M10x2"
 				(path "/28a4b045-d480-4410-adb7-fa6b33984079"
 					(reference "#PWR013")
@@
 		)
 		(instances
-			(project "MiniNDP_M10"
+			(project "MiniNDP_M10x2"
 				(path "/28a4b045-d480-4410-adb7-fa6b33984079"
 					(reference "#PWR058")
@@
 		)
 		(instances
-			(project "MiniNDP_M10"
+			(project "MiniNDP_M10x2"
 				(path "/28a4b045-d480-4410-adb7-fa6b33984079"
 					(reference "#PWR019")
@@
 		)
 		(instances
-			(project "MiniNDP_M10"
+			(project "MiniNDP_M10x2"
 				(path "/28a4b045-d480-4410-adb7-fa6b33984079"
 					(reference "#PWR07")
@@
 		)
 		(instances
-			(project "MiniNDP_M10"
+			(project "MiniNDP_M10x2"
 				(path "/28a4b045-d480-4410-adb7-fa6b33984079"
 					(reference "#PWR042")
@@
 		)
 		(instances
-			(project "MiniNDP_M10"
+			(project "MiniNDP_M10x2"
 				(path "/28a4b045-d480-4410-adb7-fa6b33984079"
 					(reference "#PWR057")
@@
 		)
 		(instances
-			(project "MiniNDP_M10"
+			(project "MiniNDP_M10x2"
 				(path "/28a4b045-d480-4410-adb7-fa6b33984079"
 					(reference "#PWR03")
@@
 		)
 		(instances
-			(project "MiniNDP_M10"
+			(project "MiniNDP_M10x2"
 				(path "/28a4b045-d480-4410-adb7-fa6b33984079"
 					(reference "DA1")
@@
 			)
 		)
-		(property "Value" "MiniNDP_Cover_M10"
+		(property "Value" "MiniNDP_Cover_M10compact2"
 			(at 138.43 183.642 0)
 			(effects
@@
 			)
 		)
-		(property "Footprint" "000_LOCAL:MiniNDP_Cover_M10"
+		(property "Footprint" "000_LOCAL:MiniNDP_Cover_M10compact2"
 			(at 139.7 187.96 0)
 			(effects
@@
 			)
 		)
-		(property "Description" "Snap cover for MiniNDP M10"
+		(property "Description" "Snap cover for MiniNDP M10c compact2 version"
 			(at 138.43 189.23 0)
 			(effects
@@
 			)
 		)
-		(property "MPN" "MiniNDP_Cover_M10.stl"
+		(property "MPN" "MiniNDP_Cover_M10compact2.stl"
 			(at 138.43 189.23 0)
 			(effects
@@
 		)
 		(instances
-			(project "MiniNDP_M10"
+			(project "MiniNDP_M10x2"
 				(path "/28a4b045-d480-4410-adb7-fa6b33984079"
 					(reference "N1")
@@
 		)
 		(instances
-			(project "MiniNDP_M10"
+			(project "MiniNDP_M10x2"
 				(path "/28a4b045-d480-4410-adb7-fa6b33984079"
 					(reference "C5")
@@
 		)
 		(instances
-			(project "MiniNDP_M10"
+			(project "MiniNDP_M10x2"
 				(path "/28a4b045-d480-4410-adb7-fa6b33984079"
 					(reference "C2")
@@
 		)
 		(instances
-			(project "MiniNDP_M10"
+			(project "MiniNDP_M10x2"
 				(path "/28a4b045-d480-4410-adb7-fa6b33984079"
 					(reference "#FLG03")
@@
 		)
 		(instances
-			(project "MiniNDP_M10"
+			(project "MiniNDP_M10x2"
 				(path "/28a4b045-d480-4410-adb7-fa6b33984079"
 					(reference "#PWR023")
@@
 		)
 		(instances
-			(project "MiniNDP_M10"
+			(project "MiniNDP_M10x2"
 				(path "/28a4b045-d480-4410-adb7-fa6b33984079"
 					(reference "#PWR06")
@@
 		)
 		(instances
-			(project "MiniNDP_M10"
+			(project "MiniNDP_M10x2"
 				(path "/28a4b045-d480-4410-adb7-fa6b33984079"
 					(reference "U3")
@@
 		)
 		(instances
-			(project "MiniNDP_M10"
+			(project "MiniNDP_M10x2"
 				(path "/28a4b045-d480-4410-adb7-fa6b33984079"
 					(reference "#PWR027")
@@
 		)
 		(instances
-			(project "MiniNDP_M10"
+			(project "MiniNDP_M10x2"
 				(path "/28a4b045-d480-4410-adb7-fa6b33984079"
 					(reference "#PWR014")
@@
 		)
 		(instances
-			(project "MiniNDP_M10"
+			(project "MiniNDP_M10x2"
 				(path "/28a4b045-d480-4410-adb7-fa6b33984079"
 					(reference "R1")
@@
 		)
 		(instances
-			(project "MiniNDP_M10"
+			(project "MiniNDP_M10x2"
 				(path "/28a4b045-d480-4410-adb7-fa6b33984079"
 					(reference "#PWR04")
@@
 		)
 		(instances
-			(project "MiniNDP_M10"
+			(project "MiniNDP_M10x2"
 				(path "/28a4b045-d480-4410-adb7-fa6b33984079"
 					(reference "C4")
@@
 		)
 		(instances
-			(project "MiniNDP_M10"
+			(project "MiniNDP_M10x2"
 				(path "/28a4b045-d480-4410-adb7-fa6b33984079"
 					(reference "#FLG02")
@@
 		)
 		(instances
-			(project "MiniNDP_M10"
+			(project "MiniNDP_M10x2"
 				(path "/28a4b045-d480-4410-adb7-fa6b33984079"
 					(reference "#PWR09")
@@
 		)
 		(instances
-			(project "MiniNDP_M10"
+			(project "MiniNDP_M10x2"
 				(path "/28a4b045-d480-4410-adb7-fa6b33984079"
 					(reference "#PWR02")
@@
 		)
 		(instances
-			(project "MiniNDP_M10"
+			(project "MiniNDP_M10x2"
 				(path "/28a4b045-d480-4410-adb7-fa6b33984079"
 					(reference "#PWR025")
@@
 		)
 		(instances
-			(project "MiniNDP_M10"
+			(project "MiniNDP_M10x2"
 				(path "/28a4b045-d480-4410-adb7-fa6b33984079"
 					(reference "J1")
@@
 		)
 		(instances
-			(project "MiniNDP_M10"
+			(project "MiniNDP_M10x2"
 				(path "/28a4b045-d480-4410-adb7-fa6b33984079"
 					(reference "C3")
@@
 		)
 		(instances
-			(project "MiniNDP_M10"
+			(project "MiniNDP_M10x2"
 				(path "/28a4b045-d480-4410-adb7-fa6b33984079"
 					(reference "#PWR032")
@@
 		)
 		(instances
-			(project "MiniNDP_M10"
+			(project "MiniNDP_M10x2"
 				(path "/28a4b045-d480-4410-adb7-fa6b33984079"
 					(reference "U4")
@@
 		)
 		(instances
-			(project "MiniNDP_M10"
+			(project "MiniNDP_M10x2"
 				(path "/28a4b045-d480-4410-adb7-fa6b33984079"
 					(reference "#PWR033")
@@
 		)
 		(instances
-			(project "MiniNDP_M10"
+			(project "MiniNDP_M10x2"
 				(path "/28a4b045-d480-4410-adb7-fa6b33984079"
 					(reference "#PWR011")
@@
 		)
 		(instances
-			(project "MiniNDP_M10"
+			(project "MiniNDP_M10x2"
 				(path "/28a4b045-d480-4410-adb7-fa6b33984079"
 					(reference "C1")
@@
 		)
 		(instances
-			(project "MiniNDP_M10"
+			(project "MiniNDP_M10x2"
 				(path "/28a4b045-d480-4410-adb7-fa6b33984079"
 					(reference "#PWR016")
