File: PCB/MiniNDP_M10c3.kicad_sch (KiCad schematic)
At the start: 14 parts, among them J1 Conn_02x20_Odd_Even, U1 AS6C8008_TSOPII, U2 HC238, U3 HC4040, U4 ABT841

Commit message: Olivetti M-10 take 3. T512 pics readme.
Parts:
- N1: value MiniNDP_Cover_M10 -> MiniNDP_Cover_M10compact2; footprint 000_LOCAL:MiniNDP_Cover_M10 -> 000_LOCAL:MiniNDP_Cover_M10compact2; MPN MiniNDP_Cover_M10.stl -> MiniNDP_Cover_M10compact2.stl
Connections:
- net A15: now also U1.27 (A10); no longer U1.23 (A14)
- net A16: now also U1.26 (A11); no longer U1.24 (A13)
- net A18: now also U1.24 (A13); no longer U1.26 (A11)
- net A19: now also U1.23 (A14); no longer U1.27 (A10)
- net AD0: now also U1.31 (Q4), U4.11 (D9); no longer U1.14 (Q3), U4.2 (D0)
- net AD1: now also U1.32 (Q5), U4.10 (D8); no longer U1.13 (Q2), U4.3 (D1)
- net AD2: now also U1.35 (Q6), U4.9 (D7); no longer U1.10 (Q1), U4.4 (D2)
- net AD3: now also U1.36 (Q7), U4.8 (D6); no longer U1.9 (Q0), U4.5 (D3)
- net AD4: now also U1.9 (Q0), U4.7 (D5); no longer U1.31 (Q4), U4.6 (D4)
- net AD5: now also U1.10 (Q1), U4.6 (D4); no longer U1.32 (Q5), U4.7 (D5)
- net AD6: now also U1.13 (Q2), U4.5 (D3); no longer U1.35 (Q6), U4.8 (D6)
- net AD7: now also U1.14 (Q3), U4.4 (D2); no longer U1.36 (Q7), U4.9 (D7)
- net BUS_A10: now also U4.2 (D0); no longer U4.11 (D9)
- net BUS_A11: now also U4.3 (D1); no longer U4.10 (D8)
Other:
- note removed: "1M for Olivetti M-10"
- title: MiniNDP_M10 -> MiniNDP_M10c2

Commit message: remove junk
Parts:
- N1: value MiniNDP_Cover_M10compact2 -> MiniNDP_Cover_M10; footprint 000_LOCAL:MiniNDP_Cover_M10compact2 -> 000_LOCAL:MiniNDP_Cover_M10; MPN MiniNDP_Cover_M10compact2.stl -> MiniNDP_Cover_M10.stl
Changed lines of the file:
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@@
 			)
 		)
-		(property "Value" "MiniNDP_Cover_M10compact2"
+		(property "Value" "MiniNDP_Cover_M10"
 			(at 138.43 183.642 0)
 			(effects
@@
 			)
 		)
-		(property "Footprint" "000_LOCAL:MiniNDP_Cover_M10compact2"
+		(property "Footprint" "000_LOCAL:MiniNDP_Cover_M10"
 			(at 139.7 187.96 0)
 			(effects
@@
 			)
 		)
-		(property "Description" "Snap cover for MiniNDP M10c compact2 version"
+		(property "Description" "Snap cover for MiniNDP M10"
 			(at 138.43 189.23 0)
 			(effects
@@
 			)
 		)
-		(property "MPN" "MiniNDP_Cover_M10compact2.stl"
+		(property "MPN" "MiniNDP_Cover_M10.stl"
 			(at 138.43 189.23 0)
 			(effects
