File: PCB/Control_Logic_Reference.kicad_sch (KiCad schematic)
At the start: 4 parts, among them U1 HC00, U2 HC08, U3 HC08, U4 HC00

Commit message: M10 cover symmetrical
Connections:
- net BLOCK: no longer U1.6
- net BYTE: no longer U1.11
- new net ~{BLOCK}: U1.6
- new net ~{BYTE}: U1.11
Other:
- note added: "BUS BUS (A) ~{YO} _A8 _A9 -> ~{BLOCK} ~{BYTE} Function L X X X X X X H X X X X X X L X X X H L H L -> L H Select BLOCK H L H H -> H L Read or Write BYTE ~{BLOCK} L: sets A0-A9 to 0, updates A10-A17 from AD0-AD7 H: latches A10-A17 ~{BYTE} L: enables SRAM for read or write H: disables SRAM, increments A0-A9 by 1"
- note removed: "BUS BUS (A) ~{YO} _A8 _A9 -> BLOCK BYTE Function L X X X X X X H X X X X X X L X X X H L H L -> L H Select BLOCK H L H H -> H L Read or Write BYTE ~{BLOCK} L: sets A0-A9 to 0, updates A10-A17 from AD0-AD7 H: latches A10-A17 ~{BYTE} L: enables SRAM for read or write H: disables SRAM, increments A0-A9 by 1"
