File: attic/PCB/MiniNDP_M10v1.kicad_pcb (KiCad board)
At the start: 2 copper layers, 60 x 34 mm, 22 parts, among them J1 Conn_02x20_Odd_Even, U1 AS6C8008_TSOPII, U2 HC238, U3 HC4040, U4 ABT841

Commit message: M10 better layout, put old M10 versions in attic
Routing:
- net /RAMRST: track 29.1 -> 29.0 mm, vias 2 -> 1
- net GND: vias 81 -> 78
