File: attic/PCB/MiniNDP_M10v2.kicad_pcb (KiCad board)
At the start: 2 copper layers, 56 x 31 mm, 22 parts, among them J1 Conn_02x20_Odd_Even, U1 AS6C8008_TSOPII, U2 HC238, U3 HC4040, U4 ABT841

Commit message: M10 better layout, put old M10 versions in attic
Parts:
- N1: value MiniNDP_Cover_M10compact -> MiniNDP_Cover_M10v2; footprint 000_LOCAL:MiniNDP_Cover_M10compact -> 000_LOCAL:MiniNDP_Cover_M10v2
Changed lines of the file:
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@@
 	(title_block
 		(title "MiniNDP")
-		(date "2026-08-12")
-		(rev "M10c_16")
+		(date "2026-08-14")
+		(rev "M10v2_18")
 		(company "Brian K. White - b.kenyon.w@gmail.com")
 		(comment 1 "github.com/bkw777/NODE_DATAPAC")
@@
 		(property ki_fp_filters "C_*")
 		(sheetname "/")
-		(sheetfile "MiniNDP_M10c.kicad_sch")
+		(sheetfile "MiniNDP_M10v2.kicad_sch")
 		(attr smd)
 		(fp_line
@@
 		(property ki_fp_filters "R_*")
 		(sheetname "/")
-		(sheetfile "MiniNDP_M10c.kicad_sch")
+		(sheetfile "MiniNDP_M10v2.kicad_sch")
 		(attr smd)
 		(fp_poly
@@
 		(property ki_fp_filters "C_*")
 		(sheetname "/")
-		(sheetfile "MiniNDP_M10c.kicad_sch")
+		(sheetfile "MiniNDP_M10v2.kicad_sch")
 		(attr smd)
 		(fp_line
@@
 		(property ki_fp_filters "DIP*24* *SO*24*")
 		(sheetname "/")
-		(sheetfile "MiniNDP_M10c.kicad_sch")
+		(sheetfile "MiniNDP_M10v2.kicad_sch")
 		(attr smd)
 		(fp_line
@@
 		(property ki_fp_filters "DIP*W7.62mm* SOIC*3.9x9.9mm*P1.27mm* TSSOP*4.4x5mm*P0.65mm*")
 		(sheetname "/")
-		(sheetfile "MiniNDP_M10c.kicad_sch")
+		(sheetfile "MiniNDP_M10v2.kicad_sch")
 		(attr smd)
 		(fp_line
@@
 		(property ki_fp_filters "DIP?16* SO*16*")
 		(sheetname "/")
-		(sheetfile "MiniNDP_M10c.kicad_sch")
+		(sheetfile "MiniNDP_M10v2.kicad_sch")
 		(attr smd)
 		(fp_line
@@
 		(embedded_fonts no)
 	)
-	(footprint "000_LOCAL:MiniNDP_Cover_M10compact"
+	(footprint "000_LOCAL:MiniNDP_Cover_M10v2"
 		(layer "F.Cu")
 		(at 151.35 102.525)
@@
 			)
 		)
-		(property "Value" "MiniNDP_Cover_M10compact"
+		(property "Value" "MiniNDP_Cover_M10v2"
 			(at 0 1.6 0)
 			(unlocked yes)
@@
 			)
 		)
-		(property "Description" "Snap cover for MiniNDP M10c compact version"
+		(property "Description" "Snap cover for MiniNDP M10v2"
 			(at 0 0 0)
 			(unlocked yes)
@@
 			)
 		)
-		(property "MPN" "MiniNDP_Cover_M10compact.stl"
+		(property "MPN" "MiniNDP_Cover_M10v2.stl"
 			(at 0 0 0)
 			(unlocked yes)
@@
 		(property ki_fp_filters "Enclosure* Housing*")
 		(sheetname "/")
-		(sheetfile "MiniNDP_M10c.kicad_sch")
+		(sheetfile "MiniNDP_M10v2.kicad_sch")
 		(attr board_only exclude_from_pos_files exclude_from_bom allow_missing_courtyard)
 		(fp_line
@@
 		)
 		(embedded_fonts no)
-		(model "${KIPRJMOD}/000_LOCAL.pretty/3dshapes/MiniNDP_Cover_M10compact.step"
+		(model "${KIPRJMOD}/000_LOCAL.pretty/3dshapes/MiniNDP_Cover_M10v2.step"
 			(offset
 				(xyz 0 0 -1.6)
@@
 		(property ki_fp_filters "SSOP*11.305x20.495mm*P1.27mm*")
 		(sheetname "/")
-		(sheetfile "MiniNDP_M10c.kicad_sch")
+		(sheetfile "MiniNDP_M10v2.kicad_sch")
 		(attr smd)
 		(fp_line
@@
 		(property ki_fp_filters "C_*")
 		(sheetname "/")
-		(sheetfile "MiniNDP_M10c.kicad_sch")
+		(sheetfile "MiniNDP_M10v2.kicad_sch")
 		(attr smd)
 		(fp_line
@@
 		(property ki_fp_filters "C_*")
 		(sheetname "/")
-		(sheetfile "MiniNDP_M10c.kicad_sch")
+		(sheetfile "MiniNDP_M10v2.kicad_sch")
 		(attr smd)
 		(fp_line
@@
 		)
 		(sheetname "/")
-		(sheetfile "MiniNDP_M10c.kicad_sch")
+		(sheetfile "MiniNDP_M10v2.kicad_sch")
 		(zone_connect 2)
 		(attr smd)
@@
 		(property ki_fp_filters "C_*")
 		(sheetname "/")
-		(sheetfile "MiniNDP_M10c.kicad_sch")
+		(sheetfile "MiniNDP_M10v2.kicad_sch")
 		(attr smd)
 		(fp_line
@@
 		(property ki_fp_filters "SOT?23*")
 		(sheetname "/")
-		(sheetfile "MiniNDP_M10c.kicad_sch")
+		(sheetfile "MiniNDP_M10v2.kicad_sch")
 		(attr smd)
 		(fp_line
@@
 		(property ki_fp_filters "Connector*:*_2x??_*")
 		(sheetname "/")
-		(sheetfile "MiniNDP_M10c.kicad_sch")
+		(sheetfile "MiniNDP_M10v2.kicad_sch")
 		(attr through_hole)
 		(fp_line
@@
 		(effects
 			(font
-				(size 1.5 1.5)
+				(size 1.5 1.4)
 				(thickness 0.15)
 			)
